File: Project2/Project2.sch (KiCad schematic (older format))
At the start: 75 parts

Commit message: Made some updates
Parts:
- added C?: 470 pF, symbol C
- added C? (x2): CP, symbol CP
- added D?: D, symbol D
- added L?: L, symbol L
- added Q?: Q_PMOS_DGS, symbol Q_PMOS_DGS
- added R? (x5): R, symbol R
- added U?: AZ34063U, symbol AZ34063U
- added U?: NCP1117-5.0_SOT223, TO_SOT_Packages_SMD:SOT-223-3Lead_TabPin2, symbol NCP1117-5.0_SOT223
- added U?: OP179GRT, TO_SOT_Packages_SMD:SOT-23-5, symbol OP179GRT
Connections:
- net +3V3: now also U?.4 (-)
- net GND: now also C?.2, C?.2, C?.2, D?.2 (A), R?.1, R?.2, U?.1 (GND), U?.4 (GND), U?.5 (V-)
- new net: R?.1, U?.1 (Switch_Collector), U?.7 (Ipk_Sense), U?.8 (Driver_Collector)
- new net: L?.1, U?.2 (Switch_Emitter)
- new net: C?.1, U?.3 (Timing_Capacitor)
- new net: R?.1, R?.2, U?.5 (Comparator_Inverting_Input)
- new net: C?.1, R?.2, U?.6 (Vcc)
- new net: C?.1, L?.2, R?.2, U?.3 (VI)
- new net: Q?.2 (G), U?.1
- new net: R?.1, R?.2, U?.3 (+)
- new net +5V: Q?.1 (D), U?.2 (V+), U?.2 (VO)
- new net Vin: R?.1

Commit message: Add files via upload
Parts:
- removed C?: 470 pF, symbol C
- removed C? (x2): CP, symbol CP
- removed D?: D, symbol D
- removed J?: Conn_02x10_Top_Bottom, symbol Conn_02x10_Top_Bottom
- removed J?: Conn_02x17_Top_Bottom, symbol Conn_02x17_Top_Bottom
- removed L?: L, symbol L
- removed Q?: Q_PMOS_DGS, symbol Q_PMOS_DGS
- removed R? (x5): R, symbol R
- removed U?: AZ34063U, symbol AZ34063U
- removed U?: NCP1117-5.0_SOT223, TO_SOT_Packages_SMD:SOT-223-3Lead_TabPin2, symbol NCP1117-5.0_SOT223
- removed U?: OP179GRT, TO_SOT_Packages_SMD:SOT-23-5, symbol OP179GRT
- added C10, C34, C35: 4.7uF, symbol C
- added C12, C19, C28, C8: 0.1uF, symbol C
- added C20: 82.0pF, symbol C
- added C25, C27: 22uF, symbol C
- added C29, C32, C6: 10uF, symbol C
- added D1: S210FA, symbol D_Schottky
- added D2: LED, symbol LED
- added L2: 10.0uH, symbol L
- added Q1: FDN304, symbol Q_PMOS_GDS
- added R1: 10k, symbol R
- added R16: 100k, symbol R
- added R17: 11.3k, symbol R
- added R29: 267k, symbol R
- added R3, R7: 0, symbol R
- added R30: 30.1k, symbol R
- added R33: 1k, symbol R
- added R5: 47.5k, symbol R
- added R6: 634, symbol R
- added U1: STMPS2141, symbol STMPS2141
- added U3: TPS54202, symbol TPS54202
- added U4: LM358, symbol LM358
- added U5: TPS7A7001, symbol TPS7A7001
- added U8: AP2114H-3.3, TO_SOT_Packages_SMD:SOT-223-3Lead_TabPin2, symbol AP1117-33-RESCUE-Project2
- C21, C23: renamed from C?; value C -> 6.0pF
- C22: renamed from C?; value C -> 4.7uF
- C24: renamed from C?; value C -> 0.1uF
- C3, C4: renamed from C?; value C -> 15pF
- L1: renamed from L?; value L -> 10uH
- gave numbers to parts that had none: 64
Connections:
- net +3V3: now also J5.1 (Pin_1), J5.2 (Pin_2), J5.3 (Pin_3), J5.37 (Pin_37), J5.38 (Pin_38), J5.39 (Pin_39), J7.1 (Pin_1), J7.37 (Pin_37), J8.10 (Pin_10), J8.11 (Pin_11), J8.12 (Pin_12), J8.13 (Pin_13), J8.14 (Pin_14), J8.15 (Pin_15), J8.16 (Pin_16), J8.9 (Pin_9), C12.1, C35.1, R1.1, R5.1, R6.1, U4.6 (-), U8.2 (VO)
- net +5V: now also J6.16 (Pin_16), J6.17 (Pin_17), J6.18 (Pin_18), J6.19 (Pin_19), J6.20 (Pin_20), J6.21 (Pin_21), J6.22 (Pin_22), J6.23 (Pin_23), J6.24 (Pin_24), J6.25 (Pin_25), J6.26 (Pin_26), J6.27 (Pin_27), J6.28 (Pin_28), J6.29 (Pin_29), J6.30 (Pin_30), C32.1, C34.1, Q1.3 (S), R29.1, R33.1, U1.5 (IN), U4.8 (V+), U5.6 (OUT), U8.3 (VI), U8.~ (EN)
- net AUX_CLK: now also J5.41 (Pin_41), J5.5 (Pin_5)
- net AVdd: now also J5.19 (Pin_19), J5.55 (Pin_55)
- net BOOT0: now also J7.42 (Pin_42), J7.6 (Pin_6)
- net GND: now also J1.2, J1.3, J6.1 (Pin_1), J6.10 (Pin_10), J6.11 (Pin_11), J6.12 (Pin_12), J6.13 (Pin_13), J6.14 (Pin_14), J6.15 (Pin_15), J6.2 (Pin_2), J6.3 (Pin_3), J6.4 (Pin_4), J6.5 (Pin_5), J6.6 (Pin_6), J6.7 (Pin_7), J6.8 (Pin_8), J6.9 (Pin_9), J8.1 (Pin_1), J8.2 (Pin_2), J8.3 (Pin_3), J8.4 (Pin_4), J8.5 (Pin_5), J8.6 (Pin_6), J8.7 (Pin_7), J8.8 (Pin_8), C10.2, C12.2, C25.2, C27.2, C28.2, C29.2, C32.2, C34.2, C35.2, C6.2, C8.2, R17.2, R30.2, U1.2 (GND), U3.1 (GND), U4.2 (-), U4.3 (+), U4.4 (V-), U5.8 (GND), U5.~ (PAD), U8.1 (GND)
- net SDO: now also J5.4 (Pin_4), J5.40 (Pin_40)
- net VBAT: now also J5.13 (Pin_13), J5.49 (Pin_49)
- net V_USB: now also C31.1, J3.1 (VBUS), Q1.2 (D)
- net Vin: now also J1.1, D1.2 (A)
- net PC0: now reaches U2.15 (PC0)
- net PC0: now also J5.15 (Pin_15), J5.51 (Pin_51)
- net PC1: now reaches U2.16 (PC1)
- net PC1: now also J5.16 (Pin_16), J5.52 (Pin_52)
- net PC2: now reaches U2.17 (PC2)
- net PC2: now also J5.17 (Pin_17), J5.53 (Pin_53)
- net PC3: now reaches U2.18 (PC3)
- net PC3: now also J5.18 (Pin_18), J5.54 (Pin_54)
- net PA0: now reaches R9.1, U2.22 (PA0-WKUP)
- net PA0: now also J5.20 (Pin_20), J5.56 (Pin_56)
- net PA1: now reaches U2.23 (PA1)
- net PA1: now also J5.21 (Pin_21), J5.57 (Pin_57)
- net PA2: now reaches R8.1, U2.24 (PA2)
- net PA2: now also J5.22 (Pin_22), J5.58 (Pin_58)
- net PA3: now reaches U2.25 (PA3)
- net PA3: now also J5.23 (Pin_23), J5.59 (Pin_59)
- net PC4: now reaches U2.32 (PC4)
- net PC4: now also J5.24 (Pin_24), J5.60 (Pin_60)
- net PC5: now reaches U2.33 (PC5)
- net PC5: now also J5.25 (Pin_25), J5.61 (Pin_61)
- net PB0: now reaches R12.2, U2.34 (PB0)
- net PB0: now also J5.26 (Pin_26), J5.62 (Pin_62)
- net PB1: now reaches U2.35 (PB1)
- net PB1: now also J5.27 (Pin_27), J5.63 (Pin_63)
- net PB2: now reaches U2.36 (PB2)
- net PB2: now also J5.28 (Pin_28), J5.64 (Pin_64)
- net PB10: now reaches U2.46 (PB10)
- net PB10: now also J5.35 (Pin_35), J5.71 (Pin_71)
- net PB11: now reaches U2.47 (PB11)
- net PB11: now also J5.36 (Pin_36), J5.72 (Pin_72)
- net PB12: now reaches U2.51 (PB12)
- net PB12: now also J7.36 (Pin_36), J7.72 (Pin_72)
- net PB13: now reaches U2.52 (PB13)
- net PB13: now also J7.35 (Pin_35), J7.71 (Pin_71)
- net PB14: now reaches R15.2, U2.53 (PB14)
- net PB14: now also J7.34 (Pin_34), J7.70 (Pin_70)
- net PB15: now reaches U2.54 (PB15)
- net PB15: now also J7.33 (Pin_33), J7.69 (Pin_69)
- net PC6: now reaches U2.63 (PC6)
- net PC6: now also J7.24 (Pin_24), J7.60 (Pin_60)
- net PC7: now reaches U2.64 (PC7)
- net PC7: now also J7.23 (Pin_23), J7.59 (Pin_59)
- net PA8: now reaches U2.67 (PA8)
- net PA8: now also J7.22 (Pin_22), J7.58 (Pin_58)
- net at CR1.1, J2.1 (VBUS), U2.68 (PA9): now also C10.1, U1.1 (OUT)
- net PA13: now reaches U2.72 (PA13)
- net PA13: now also J7.21 (Pin_21), J7.57 (Pin_57)
- net PA14: now reaches U2.76 (PA14)
- net PA14: now also J7.20 (Pin_20), J7.56 (Pin_56)
- net JTDI: now reaches U2.77 (PA15)
- net JTDI: now also J7.19 (Pin_19), J7.55 (Pin_55)
- net JTDO: now reaches U2.89 (PB3)
- net JTDO: now also J7.11 (Pin_11), J7.47 (Pin_47)
- net NJTRST: now reaches U2.90 (PB4)
- net NJTRST: now also J7.10 (Pin_10), J7.46 (Pin_46)
- net PB5: now reaches U2.91 (PB5)
- net PB5: now also J7.45 (Pin_45), J7.9 (Pin_9)
- net PB6: now reaches U2.92 (PB6)
- net PB6: now also J7.44 (Pin_44), J7.8 (Pin_8)
- net PB7: now reaches R14.2, U2.93 (PB7)
- net PB7: now also J7.43 (Pin_43), J7.7 (Pin_7)
- net PB8: now reaches U2.95 (PB8)
- net PB8: now also J7.41 (Pin_41), J7.5 (Pin_5)
- net PB9: now reaches U2.96 (PB9)
- net PB9: now also J7.4 (Pin_4), J7.40 (Pin_40)
- net PE2: now reaches U2.1 (PE2)
- net PE2: now also J5.44 (Pin_44), J5.8 (Pin_8)
- net PE3: now reaches U2.2 (PE3)
- net PE3: now also J5.45 (Pin_45), J5.9 (Pin_9)
- net PE4: now reaches U2.3 (PE4)
- net PE4: now also J5.10 (Pin_10), J5.46 (Pin_46)
- net PE5: now reaches U2.4 (PE5)
- net PE5: now also J5.11 (Pin_11), J5.47 (Pin_47)
- net PE11: now reaches U2.41 (PE11)
- net PE11: now also J5.30 (Pin_30), J5.66 (Pin_66)
- net PE12: now reaches U2.42 (PE12)
- net PE12: now also J5.31 (Pin_31), J5.67 (Pin_67)
- net PE13: now reaches U2.43 (PE13)
- net PE13: now also J5.32 (Pin_32), J5.68 (Pin_68)
- net PE14: now reaches U2.44 (PE14)
- net PE14: now also J5.33 (Pin_33), J5.69 (Pin_69)
- net PE15: now reaches U2.45 (PE15)
- net PE15: now also J5.34 (Pin_34), J5.70 (Pin_70)
- net PE6: now reaches U2.5 (PE6)
- net PE6: now also J5.12 (Pin_12), J5.48 (Pin_48)
- net PD8: now reaches U2.55 (PD8)
- net PD8: now also J7.32 (Pin_32), J7.68 (Pin_68)
- net PD9: now reaches U2.56 (PD9)
- net PD9: now also J7.31 (Pin_31), J7.67 (Pin_67)
- net PD10: now reaches U2.57 (PD10)
- net PD10: now also J7.30 (Pin_30), J7.66 (Pin_66)
- net PD11: now reaches U2.58 (PD11)
- net PD11: now also J7.29 (Pin_29), J7.65 (Pin_65)
- net PD12: now reaches U2.59 (PD12)
- net PD12: now also J7.28 (Pin_28), J7.64 (Pin_64)
- net PD13: now reaches U2.60 (PD13)
- net PD13: now also J7.27 (Pin_27), J7.63 (Pin_63)
- net PD14: now reaches U2.61 (PD14)
- net PD14: now also J7.26 (Pin_26), J7.62 (Pin_62)
- net PD15: now reaches U2.62 (PD15)
- net PD15: now also J7.25 (Pin_25), J7.61 (Pin_61)
- net PD0: now reaches U2.81 (PD0)
- net PD0: now also J7.18 (Pin_18), J7.54 (Pin_54)
- net PD1: now reaches U2.82 (PD1)
- net PD1: now also J7.17 (Pin_17), J7.53 (Pin_53)
- net PD3: now reaches U2.84 (PD3)
- net PD3: now also J7.16 (Pin_16), J7.52 (Pin_52)
- net OTG_FS_OverCurrent: now reaches U2.85 (PD4)
- net OTG_FS_OverCurrent: now also J7.15 (Pin_15), J7.51 (Pin_51), R7.1
- net OTG_FS_PWR_SW: now reaches U2.86 (PD5)
- net OTG_FS_PWR_SW: now also J7.14 (Pin_14), J7.50 (Pin_50), R3.1
- net PD6: now reaches U2.87 (PD6)
- net PD6: now also J7.13 (Pin_13), J7.49 (Pin_49)
- net PD7: now reaches U2.88 (PD7)
- net PD7: now also J7.12 (Pin_12), J7.48 (Pin_48)
- net PE0: now reaches U2.97 (PE0)
- net PE0: now also J7.3 (Pin_3), J7.39 (Pin_39)
- net PE1: now reaches U2.98 (PE1)
- net PE1: now also J7.2 (Pin_2), J7.38 (Pin_38)
- net NRST: now reaches C16.2, SW1.1, SW1.3, U2.14 (NRST)
- net NRST: now also J5.14 (Pin_14), J5.50 (Pin_50)
- net PE10: now reaches J5.29 (Pin_29)
- net PE10: now also J5.65 (Pin_65)
- net CBUS3: now reaches J5.42 (Pin_42)
- net CBUS3: now also J5.6 (Pin_6), U7.16 (CBUS3)
- net CBUS0: now reaches J5.43 (Pin_43)
- net CBUS0: now also J5.7 (Pin_7), U7.15 (CBUS0)
- new net: C6.1, C8.1, D1.1 (K), U3.3 (VIN)
- new net: C19.1, L2.1, U3.2 (SW)
- new net: C20.2, R16.2, R17.1, U3.4 (FB)
- new net: C19.2, U3.6 (BOOT)
- new net: C20.1, C25.1, C27.1, C28.1, C29.1, L2.2, R16.1, U5.2 (EN), U5.3 (IN)
- new net: R29.2, R30.1, U5.7 (FB)
- new net: Q1.1 (G), U4.7
- new net: R33.2, U4.5 (+)
- new net: D2.1 (K), R5.2, R7.2, U1.3 (FAULT)
- new net: R1.2, R3.2, U1.4 (EN)
- new net: D2.2 (A), R6.2
Other:
- moved on the sheet: C13, C35, J1, J5, J6, J7, J8, R15, R8, U6

Commit message: Updated project 2
Parts:
- removed R33: 1k, symbol R
- removed R8: 0, symbol R
- added D7: +5V Pwr (blue), symbol LED
- added D8, D9: Vin Pwr (blue), symbol LED
- added R20: 11.3k, symbol R
- added R21: 47.5k, symbol R
- added R36: 634, symbol R
- added R37, R38: 1k, symbol R
- added unit 4 of U2
- added unit 5 of U2
- added unit 6 of U2
- renumbered C11 to C10, C12 to C11, C10 to C12, C17 to C15, C15 to C16, C16 to C17, C22 to C20, C20 to C21, C24 to C22, C21 to C23, C25 to C24, C27 to C25, C23 to C26, C26 to C27, C33 to C31, C31 to C32, C34 to C33, C32 to C34, C34 to C36, C35 to C37, R3 to R1, R11 to R10, R16 to R11, R17 to R12, R12 to R13, R13 to R14, R14 to R15, R15 to R16, R18 to R17, R20 to R18, R31 to R23, R32 to R24, R21 to R25, R29 to R26, R30 to R27, R24 to R28, R25 to R29, R1 to R3, R26 to R30, R23 to R31, R27 to R32, R28 to R33, R9 to R8, R10 to R9
Connections:
- net labels added: Vin_6V, Vsense
- net labels removed: PE10, SCLK, SDI, SDO, WKUP_2, nCS
- wire segments 570 -> 787
- no-connect marks 0 -> 6
Other:
- note removed: "Diff Pair!"
- moved on the sheet: C12, C14, C15, C20, C22, C23, C26, C27, C30, C31, C32, C33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
